File: PCB/toern_revG/toern_revF_kicad_pcb.kicad_pcb (KiCad board)
At the start: 4 copper layers, 160 x 71 mm, 92 parts, among them J1 AudioJack3_Switch, J10 Conn_01x02, J11 Conn_01x05, J11.5 Conn_01x05, J12 Conn_01x05, J13 Conn_01x05, J14 Conn_01x05, J15 Conn_01x05, J16 BATTERY, J17 AudioJack3_Ground, J3 AudioJack3_Ground, J4 USB_C_Receptacle_USB2.0, J5 AudioJack3_Switch, J6 AudioJack3_Switch, J7 AudioJack3_Switch, J8 Micro_SD_Card, J9 Conn_01x03, Q1 DMG3415, SW1 EG2219, U1 SPX3819M5-L-3-3, U10 01x05 Connector_PinSocket_2.5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, U11 01x05 Connector_PinSocket_2.5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, U12 01x05 Connector_PinSocket_2.5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, U13 PAM8403D, U2 SPX3819M5-L-1-8, U3 SGTL5000XNBA3, U4 TLP2361V4_E, U5 74LVC2G14, U6 Teensy4.1, U7 SPX3819M5-L-3-3, U8 MCP73831-3-OT, U9 01x05 Connector_PinSocket_2.5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

Commit message: more fixes
Parts:
- removed C27, C28: 0.47uF, Capacitor_SMD:C_0603_1608Metric
- removed C29: 0.1uF, Capacitor_SMD:C_0603_1608Metric
- removed C30, C31: 1uF, Capacitor_SMD:C_0603_1608Metric
- removed J10: Conn_01x02, Connector_JST:JST_PH_B2B-PH-K_1x02_P2.00mm_Vertical
- removed J17: AudioJack3_Ground, Connector_Audio:Jack_3.5mm_CUI_SJ1-3533NG_Horizontal_CircularHoles
- removed LOGOOPENHARDWARE: OSHW-Logo2_7.3x6mm_SilkScreen, Symbol:OSHW-Logo2_7.3x6mm_SilkScreen
- removed R21, R22: 20k, Resistor_SMD:R_0603_1608Metric
- removed REF** (x2): C21081137, Connector_PinSocket_2.54mm:PinSocket_1x24_P2.54mm_Vertical
- removed U13: PAM8403D, Package_SO:SOIC-16_3.9x9.9mm_P1.27mm
- added J2: CUI_SJ2-35863B1-SMT-TR, myLibKicad:CUI_SJ2-35863B1-SMT-TR, F.Cu at (185.0, 90.0)
- J3: value AudioJack3_Ground -> CUI_SJ2-35863B1-SMT-TR; footprint Connector_Audio:Jack_3.5mm_CUI_SJ1-3533NG_Horizontal_CircularHoles -> myLibKicad:CUI_SJ2-35863B1-SMT-TR
- R15, R19: footprint Resistor_SMD:R_0603_1608Metric -> Resistor_SMD:R_0805_2012Metric
- moved MK1 22.8 mm to (106.1, 88.5), turned to 0 degrees
- moved R11 18.6 mm to (111.0, 84.8)
- moved R8 15.9 mm to (184.8, 83.5), turned to 180 degrees
- moved J3 12.5 mm to (184.9, 77.0), turned to 180 degrees
- moved R7 9.65 mm to (187.5, 70.5), turned to 0 degrees
- moved R20 2.12 mm to (140.0, 30.5)
Connections:
- J13 pad 4: 6_OUT1D -> +3.3V
- J13 pad 5: 39_MISO1_OUT1A -> GND
- R6 pad 2: Net-(J3-PadR) -> Net-(J2-Pad3)
- R7 pad 2: Net-(J17-PadT) -> Net-(J3-Pad2)
- R8 pad 1: Net-(J17-PadR) -> Net-(J3-Pad3)
Routing:
- net 30_CRX3: track 130.8 -> 0.00 mm, vias 2 -> 0
- net 39_MISO1_OUT1A: track 82.4 -> 0.00 mm, vias 2 -> 0
- net Net-(J2-Pad3): track 0.00 -> 78.1 mm
- net Net-(J3-PadR): track 71.1 -> 0.00 mm
- net 6_OUT1D: track 63.4 -> 0.00 mm, vias 1 -> 0
- net Net-(U3-HP_L): track 134.7 -> 86.6 mm
- net Net-(U3-HP_R): track 126.1 -> 91.1 mm, vias 3 -> 2
- net +5V: track 504.2 -> 473.6 mm, vias 2 -> 1
- net GND: track 101.7 -> 72.9 mm, vias 60 -> 53
- net Net-(J10-Pin_1): track 19.5 -> 0.00 mm
- net Net-(J17-PadT): track 19.0 -> 0.00 mm
- net MICBIAS: track 40.3 -> 57.0 mm
- net Net-(J10-Pin_2): track 15.9 -> 0.00 mm
- net Net-(MK1-+): track 50.1 -> 37.3 mm
- net Net-(U13-VREF): track 12.8 -> 0.00 mm
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Other:
- board text added: "MIDIIN"
- board text added: "MIDIOUT"
- board text added: "V1.2"
- board text added: "made by jpk in Hamburg, st.pauli. find me online at: www.toern.live"
- board text added: "shoutout to pjrc, arduino, duppa and makerhafen HH"
- board text added: "{dblquote}Weisst du was ich manchmal denke? Es müsste immer Musik da sein. Bei allem was du machst. Und wenns so richtig scheisse ist, dann ist wenigstens noch die Musik da. Und an der Stelle wo es am allerschönsten ist, da müsste die Platte springen - und du hörst immer nur diesen einen Moment.{dblquote} (Absolute Giganten)"
- board text removed: "(I2S2-5V)"
- board text removed: "CC BY-NC 4.0"
- board text removed: "MIDI-IN"
- board text removed: "MIDI-OUT"
- board text removed: "SPEAKER"
- board text removed: "U10"
- board text removed: "U12"
- board text removed: "U9"
- board text removed: "made in st.pauli by jan kuntoff/SP_ctrl V2.0 - 03/26 www.toern.live"
- board text removed: "{dblquote}Weisst du was ich manchmal denke? Es müsste immer Musik da sein. Bei allem was du machst. Und wenns so richtig scheisse ist, dann ist wenigstens noch die Musik da. Und an der Stelle wo es am aller- schönsten ist, da müsste die Platte springen - und du hörst immer nur diesen einen Moment.{dblquote} (Absolute Giganten)"
