File: PCB/toern_revG/toern_revG.kicad_pcb (KiCad board)
At the start: 4 copper layers, 160 x 71 mm, 108 parts, among them IC1 BQ24075TRGTR, J1 AudioJack3_Switch, J10 Conn_01x02, J11 Conn_01x05, J11.5 Conn_01x05, J12 Conn_01x05, J13 Conn_01x05, J14 Conn_01x05, J15 Conn_01x05, J16 Conn_01x02, J17 AudioJack3_Ground, J18 Conn_01x05_Socket, J19 Conn_01x05_Socket, J2 Conn_01x05_Socket, J20 Conn_01x05_Socket, J21 Conn_01x05_Socket, J22 Conn_01x05_Socket, J23 Conn_01x05_Socket, J24 Conn_01x05_Socket, J3 AudioJack3_Ground, J4 USB_C_Receptacle_USB2.0, J5 AudioJack3_Switch, J6 AudioJack3_Switch, J7 AudioJack3_Switch, J8 Micro_SD_Card, J9 Conn_01x03, U1 SPX3819M5-L-3-3, U13 PAM8403D, U2 SPX3819M5-L-1-8, U3 SGTL5000XNBA3, U4 TLP2361V4_E, U5 74LVC2G14, U6 Teensy4.1, U7 SPX3819M5-L-3-3, U8 TPS22918DBVR

Commit message: changed R14 and R18 to 200Ohm/49.9k
Co-authored-by: Cursor <cursoragent@cursor.com>
Parts:
- R14: value 10k -> 49.9k
- R18: value 47k -> 200
Changed lines of the file:
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@@
 			)
 		)
-		(property "Value" "47k"
+		(property "Value" "200"
 			(at 0 1.17 90)
 			(layer "F.Fab")
@@
 			)
 		)
-		(property "lcsc#" "C25792"
+		(property "lcsc#" "C25087"
 			(at 0 0 270)
 			(unlocked yes)
@@
 			)
 		)
-		(property "lscs#" "C25792 "
+		(property "lscs#" "C25087"
 			(at 0 0 270)
 			(unlocked yes)
@@
 			)
 		)
-		(property "Value" "10k"
+		(property "Value" "49.9k"
 			(at 0 1.17 90)
 			(layer "F.Fab")
@@
 			)
 		)
-		(property "lcsc#" "C25744"
+		(property "lcsc#" "C100457"
 			(at 0 0 270)
 			(unlocked yes)
