File: PCB/toern_revG/toern_revG.kicad_sch (KiCad schematic)
At the start: 113 parts, among them IC1 BQ24075TRGTR, J1 AudioJack3_Switch, J10 Conn_01x02, J11 Conn_01x05, J11.5 Conn_01x05, J12 Conn_01x05, J13 Conn_01x05, J14 Conn_01x05, J15 Conn_01x05, J16 Conn_01x02, J17 AudioJack3_Ground, J18 Conn_01x05_Socket, J19 Conn_01x05_Socket, J2 Conn_01x05_Socket, J20 Conn_01x05_Socket, J21 Conn_01x05_Socket, J22 Conn_01x05_Socket, J23 Conn_01x05_Socket, J24 Conn_01x05_Socket, J3 AudioJack3_Ground, J4 USB_C_Receptacle_USB2.0, J5 AudioJack3_Switch, J6 AudioJack3_Switch, J7 AudioJack3_Switch, J8 Micro_SD_Card, J9 Conn_01x03, U1 SPX3819M5-L-3-3, U10 01x05 Connector_PinSocket_2.5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, U11 01x05 Connector_PinSocket_2.5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, U12 01x05 Connector_PinSocket_2.5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, U13 PAM8403D, U2 SPX3819M5-L-1-8, U3 SGTL5000XNBA3, U4 TLP2361V4_E, U5 74LVC2G14, U6 Teensy4.1, U7 SPX3819M5-L-3-3, U8 TPS22918DBVR, U9 01x05 Connector_PinSocket_2.5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

Commit message: changed R14 and R18 to 200Ohm/49.9k
Co-authored-by: Cursor <cursoragent@cursor.com>
Parts:
- R14: value 10k -> 49.9k; lcsc# C25744 -> C100457
- R18: value 47k -> 200; lcsc# C25792 -> C25087
