File: PCB/toern_revH/toern_revH.kicad_pcb (KiCad board)
At the start: 4 copper layers, 160 x 71 mm, 130 parts, among them CN1 YZP0354-20100-01, CN2 YZP0354-20100-01, IC1 BQ24075TRGTR, J1 AudioJack3_Switch, J10 Conn_01x02, J11 Conn_01x05, J11.5 Conn_01x05, J12 Conn_01x05, J13 Conn_01x05, J14 Conn_01x05, J15 Conn_01x05, J16 Conn_01x02, J17 AudioJack3_Ground, J18 Conn_01x05_Socket, J19 Conn_01x05_Socket, J2 Conn_01x05_Socket, J20 Conn_01x05_Socket, J21 Conn_01x05_Socket, J22 Conn_01x05_Socket, J23 Conn_01x05_Socket, J24 Conn_01x05_Socket, J25 Conn_01x02, J26 Conn_01x02, J27 Conn_01x02, J28 929870-01-12-RA, J29 929870-01-12-RA, J3 AudioJack3_Ground, J30 929870-01-12-RA, J31 929870-01-12-RA, J4 USB_C_Receptacle_USB2.0, J5 AudioJack3_Switch, J6 AudioJack3_Switch, J7 AudioJack3_Switch, J8 Micro_SD_Card, J9 Conn_01x03, U1 SPX3819M5-L-3-3, U13 PAM8403D, U14 74LVC1G17, U15 74AHCT1G125, U16 74AHCT1G125, U2 SPX3819M5-L-1-8, U3 SGTL5000XNBA3, U4 TLP2361V4_E, U5 74LVC2G14, U6 Teensy4.1, U7 SPX3819M5-L-3-3, U8 TPS22918DBVR

Commit message: better info routes for buyers
Co-authored-by: Cursor <cursoragent@cursor.com>
Other:
- board text added: "by warft_labs V3.0 - 08/26 www.toern.live"
- board text removed: "made in st.pauli by warft_labs V3.0 - 08/26 www.toern.live"
Changed lines of the file:
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@@
 		)
 	)
-	(gr_text "made in st.pauli \nby warft_labs\nV3.0  - 08/26\nwww.toern.live\n"
+	(gr_text "\nby warft_labs\nV3.0  - 08/26\nwww.toern.live\n"
 		(at 97.5 85 0)
 		(layer "F.SilkS")
@@
 			(justify left top)
 		)
-		(render_cache "made in st.pauli \nby warft_labs\nV3.0  - 08/26\nwww.toern.live\n"
-			0
+		(render_cache "\nby warft_labs\nV3.0  - 08/26\nwww.toern.live\n" 0
 			(polygon
 				(pts
-					(xy 97.577403 85.027956
-					) (xy 97.873993 85.027956) (xy 98.006132 85.974192) (xy 98.009924 85.974192) (xy 98.142144 85.027956)
-					(xy 98.438652 85.027956) (xy 98.438652 86.35) (xy 98.242217 86.35) (xy 98.242217 85.349028) (xy 98.238507 85.349028)
-					(xy 98.08741 86.35) (xy 97.913643 86.35) (xy 97.762545 85.349028) (xy 97.758753 85.349028) (xy 97.758753 86.35)
-					(xy 97.577403 86.35)
-				)
-			)
-			(polygon
-				(pts
-					(xy 99.250277 86.35) (xy 99.042466 86.35) (xy 99.004713 86.087454) (xy 99.004713 86.091246) (xy 98.768627 86.091246)
-					(xy 98.730874 86.35) (xy 98.53823 86.35) (xy 98.609598 85.911791) (xy 98.793192 85.911791) (xy 98.980148 85.911791)
-					(xy 98.887659 85.258353) (xy 98.883867 85.258353) (xy 98.793192 85.911791) (xy 98.609598 85.911791)
-					(xy 98.753542 85.027956) (xy 99.034965 85.027956)
-				)
-			)
-			(polygon
-				(pts
-					(xy 99.744808 85.033925) (xy 99.807578 85.050471) (xy 99.85847 85.076271) (xy 99.899594 85.111047)
-					(xy 99.931774 85.154444) (xy 99.955904 85.207983) (xy 99.971462 85.273813) (xy 99.97708 85.354634)
-					(xy 99.97708 86.023239) (xy 99.971461 86.104105) (xy 99.955901 86.169962) (xy 99.93177 86.223512)
-					(xy 99.899594 86.266908) (xy 99.85847 86.301684) (xy 99.807578 86.327484) (xy 99.744808 86.34403)
-					(xy 99.667383 86.35) (xy 99.35002 86.35) (xy 99.35002 86.161148) (xy 99.557831 86.161148) (xy 99.663591 86.161148)
-					(xy 99.709789 86.153154) (xy 99.741902 86.130978) (xy 99.761519 86.0946) (xy 99.769351 86.032719)
-					(xy 99.769351 85.345236) (xy 99.761516 85.283369) (xy 99.741902 85.24706) (xy 99.709782 85.22482)
-					(xy 99.663591 85.216807) (xy 99.557831 85.216807) (xy 99.557831 86.161148) (xy 99.35002 86.161148)
-					(xy 99.35002 85.027956) (xy 99.667383 85.027956)
-				)
-			)
-			(polygon
-				(pts
-					(xy 100.116308 85.027956) (xy 100.682945 85.027956) (xy 100.682945 85.216807) (xy 100.324118 85.216807)
-					(xy 100.324118 85.566236) (xy 100.609251 85.566236) (xy 100.609251 85.755088) (xy 100.324118 85.755088)
-					(xy 100.324118 86.161148) (xy 100.682945 86.161148) (xy 100.682945 86.35) (xy 100.116308 86.35)
-				)
-			)
-			(polygon
-				(pts
-					(xy 101.104172 85.027956) (xy 101.311983 85.027956) (xy 101.311983 86.35) (xy 101.104172 86.35)
-				)
-			)
-			(polygon
-				(pts
-					(xy 101.466873 85.027956) (xy 101.727523 85.027956) (xy 101.929646 85.819303) (xy 101.933438 85.819303)
-					(xy 101.933438 85.027956) (xy 102.118497 85.027956) (xy 102.118497 86.35) (xy 101.905081 86.35)
-					(xy 101.655807 85.384886) (xy 101.652015 85.384886) (xy 101.652015 86.35) (xy 101.466873 86.35)
-				)
-			)
-			(polygon
-				(pts
-					(xy 102.844888 86.368876) (xy 102.769716 86.3628) (xy 102.708174 86.345857) (xy 102.657676 86.319222)
-					(xy 102.616304 86.282982) (xy 102.584059 86.238214) (xy 102.55995 86.183638) (xy 102.544468 86.117241)
-					(xy 102.5389 86.036511) (xy 102.5389 85.960921) (xy 102.735336 85.960921) (xy 102.735336 86.051596)
-					(xy 102.743297 86.111949) (xy 102.76383 86.149749) (xy 102.79574 86.171937) (xy 102.842992 86.180025)
-					(xy 102.890743 86.171727) (xy 102.923198 86.148866) (xy 102.942794 86.1115) (xy 102.950648 86.047804)
-					(xy 102.940904 85.968585) (xy 102.912812 85.901487) (xy 102.864456 85.837816) (xy 102.77309 85.7494)
-					(xy 102.690123 85.670057) (xy 102.631932 85.602325) (xy 102.593635 85.544474) (xy 102.565636 85.481672)
-					(xy 102.548558 85.413138) (xy 102.542692 85.337653) (xy 102.548327 85.259102) (xy 102.56407 85.193954)
-					(xy 102.588745 85.139861) (xy 102.621992 85.094973) (xy 102.664225 85.058633) (xy 102.715368 85.031968)
-					(xy 102.777263 85.015049) (xy 102.852389 85.008996) (xy 102.926582 85.015067) (xy 102.987332 85.032001)
-					(xy 103.037205 85.058652) (xy 103.078088 85.094973) (xy 103.109915 85.139641) (xy 103.133748 85.194175)
-					(xy 103.14907 85.260602) (xy 103.154585 85.341444) (xy 103.154585 85.396179) (xy 102.958232 85.396179)
-					(xy 102.958232 85.328255) (xy 102.950686 85.266129) (xy 102.931771 85.22909) (xy 102.900303 85.206185)
-					(xy 102.854285 85.19793) (xy 102.808893 85.205819) (xy 102.778096 85.227548) (xy 102.758172 85.264774)
-					(xy 102.750421 85.324463) (xy 102.760049 85.393652) (xy 102.789164 85.45858) (xy 102.838207 85.521519)
-					(xy 102.929875 85.609596) (xy 103.013835 85.689202) (xy 103.071869 85.757246) (xy 103.109247 85.815511)
-					(xy 103.135954 85.878952) (xy 103.152572 85.950827) (xy 103.158377 86.032719) (xy 103.15262 86.114269)
-					(xy 103.1366 86.181384) (xy 103.111607 86.236617) (xy 103.078088 86.281993) (xy 103.035378 86.318705)
-					(xy 102.983629 86.345653) (xy 102.920971 86.362756)
-				)
-			)
-			(polygon
-				(pts
-					(xy 103.440211 85.216807) (xy 103.223003 85.216807) (xy 103.223003 85.027956) (xy 103.865148 85.027956)
-					(xy 103.865148 85.216807) (xy 103.64794 85.216807) (xy 103.64794 86.35) (xy 103.440211 86.35)
-				)
-			)
-			(polygon
-				(pts
-					(xy 103.827724 86.149772) (xy 104.027951 86.149772) (xy 104.027951 86.35) (xy 103.827724 86.35)
-				)
-			)
-			(polygon
-				(pts
-					(xy 104.565969 85.033926) (xy 104.628765 85.050474) (xy 104.679669 85.076275) (xy 104.720792 85.111047)
-					(xy 104.752972 85.154444) (xy 104.777102 85.207983) (xy 104.79266 85.273813) (xy 104.798278 85.354634)
-					(xy 104.798278 85.484959) (xy 104.792659 85.565825) (xy 104.777099 85.631682) (xy 104.752969 85.685232)
-					(xy 104.720792 85.728627) (xy 104.679669 85.7634) (xy 104.628765 85.789201) (xy 104.565969 85.805748)
-					(xy 104.488499 85.811719) (xy 104.390322 85.811719) (xy 104.390322 86.35) (xy 104.182511 86.35)
-					(xy 104.182511 85.622867) (xy 104.390322 85.622867) (xy 104.488499 85.622867) (xy 104.534615 85.615237)
-					(xy 104.564996 85.594593) (xy 104.583067 85.560021) (xy 104.590467 85.49823) (xy 104.590467 85.341444)
-					(xy 104.583064 85.279667) (xy 104.564996 85.245164) (xy 104.534607 85.224456) (xy 104.488499 85.216807)
-					(xy 104.390322 85.216807) (xy 104.390322 85.622867) (xy 104.182511 85.622867) (xy 104.182511 85.027956)
-					(xy 104.488499 85.027956)
-				)
-			)
-			(polygon
-				(pts
-					(xy 105.503236 86.35) (xy 105.295425 86.35) (xy 105.257671 86.087454) (xy 105.257671 86.091246)
-					(xy 105.021586 86.091246) (xy 104.983832 86.35) (xy 104.791189 86.35) (xy 104.862557 85.911791)
-					(xy 105.046151 85.911791) (xy 105.233107 85.911791) (xy 105.140618 85.258353) (xy 105.136826 85.258353)
-					(xy 105.046151 85.911791) (xy 104.862557 85.911791) (xy 105.006501 85.027956) (xy 105.287924 85.027956)
-				)
-			)
-			(polygon
-				(pts
-					(xy 105.901218 86.368876) (xy 105.826086 86.362829) (xy 105.764188 86.345924) (xy 105.713048 86.319283)
-					(xy 105.67082 86.282982) (xy 105.637713 86.238088) (xy 105.613027 86.183463) (xy 105.597205 86.117109)
-					(xy 105.591521 86.036511) (xy 105.591521 85.027956) (xy 105.799249 85.027956) (xy 105.799249 86.051596)
-					(xy 105.807061 86.113485) (xy 105.826617 86.149855) (xy 105.858797 86.172034) (xy 105.90501 86.180025)
-					(xy 105.951279 86.172028) (xy 105.983402 86.149855) (xy 106.002958 86.113485) (xy 106.01077 86.051596)
-					(xy 106.01077 85.027956) (xy 106.210997 85.027956) (xy 106.210997 86.036511) (xy 106.205308 86.117103)
-					(xy 106.189471 86.183455) (xy 106.16476 86.238083) (xy 106.131615 86.282982) (xy 106.089387 86.319283)
-					(xy 106.038247 86.345924) (xy 105.97635 86.362829)
-				)
-			)
-			(polygon
-				(pts
-					(xy 106.358715 85.027956) (xy 106.566526 85.027956) (xy 106.566526 86.161148) (xy 106.908371 86.161148)
-					(xy 106.908371 86.35) (xy 106.358715 86.35)
-				)
-			)
-			(polygon
-				(pts
-					(xy 107.007619 85.027956) (xy 107.21543 85.027956) (xy 107.21543 86.35) (xy 107.007619 86.35)
-				)
-			)
-			(polygon
-				(pts
